File: pcb/sunrise.kicad_sch (KiCad schematic)
At the start: 17 parts, among them J1 Conn_01x15_Female, J2 Conn_01x15_Female, J3 Conn_01x04_Female, J4 Conn_01x02_Female, Q1 TSM2302CX, Q2 TSM2302CX, Q3 TSM2302CX, U1 MCP1703A-5002_SOT223, U2 TSOP312xx

Commit message: Final layout
Parts:
- added R? (x2): 10k, Resistor_SMD:R_0805_2012Metric, symbol Device:R
- added SW?: SW_SPDT, MattisLib:SS 13PLP, symbol Switch:SW_SPDT
Connections:
- net +3.3V: now also R?.1
- net GND: now also R?.1
- net RED_IO: now also J1.2 (Pin_2); no longer J1.1 (Pin_1)
- new net: R?.2, SW?.1 (A)
- new net: R?.2, SW?.3 (C)
- new net ALARM_EN: J1.1 (Pin_1), SW?.2 (B)
Changed lines of the file:
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@@
   (junction (at 44.45 80.01) (diameter 0) (color 0 0 0 0)
   )
+  (wire (pts (xy 208.28 104.14) (xy 214.63 104.14))
+    (stroke (width 0) (type default) (color 0 0 0 0))
+  )
   (wire (pts (xy 81.28 33.02) (xy 124.46 33.02))
     (stroke (width 0) (type default) (color 0 0 0 0))
@@
     (stroke (width 0) (type default) (color 0 0 0 0))
   )
+  (wire (pts (xy 179.07 109.22) (xy 186.69 109.22))
+    (stroke (width 0) (type default) (color 0 0 0 0))
+  )
   (wire (pts (xy 104.14 57.15) (xy 104.14 59.69))
     (stroke (width 0) (type default) (color 0 0 0 0))
@@
     (stroke (width 0) (type default) (color 0 0 0 0))
   )
+  (wire (pts (xy 198.12 106.68) (xy 198.12 109.22))
+    (stroke (width 0) (type default) (color 0 0 0 0))
+  )
   (wire (pts (xy 124.46 33.02) (xy 124.46 40.64))
     (stroke (width 0) (type default) (color 0 0 0 0))
@@
     (stroke (width 0) (type default) (color 0 0 0 0))
   )
+  (wire (pts (xy 194.31 99.06) (xy 198.12 99.06))
+    (stroke (width 0) (type default) (color 0 0 0 0))
+  )
   (wire (pts (xy 20.32 144.78) (xy 30.48 144.78))
     (stroke (width 0) (type default) (color 0 0 0 0))
@@
     (stroke (width 0) (type default) (color 0 0 0 0))
   )
+  (wire (pts (xy 198.12 109.22) (xy 194.31 109.22))
+    (stroke (width 0) (type default) (color 0 0 0 0))
+  )
   (wire (pts (xy 140.97 45.72) (xy 142.24 45.72))
     (stroke (width 0) (type default) (color 0 0 0 0))
@@
     (stroke (width 0) (type default) (color 0 0 0 0))
   )
+  (wire (pts (xy 198.12 99.06) (xy 198.12 101.6))
+    (stroke (width 0) (type default) (color 0 0 0 0))
+  )
   (wire (pts (xy 151.13 45.72) (xy 154.94 45.72))
     (stroke (width 0) (type default) (color 0 0 0 0))
@@
     (stroke (width 0) (type default) (color 0 0 0 0))
   )
+  (wire (pts (xy 63.5 109.22) (xy 67.31 109.22))
+    (stroke (width 0) (type default) (color 0 0 0 0))
+  )
+  (wire (pts (xy 179.07 99.06) (xy 186.69 99.06))
+    (stroke (width 0) (type default) (color 0 0 0 0))
+  )
   (wire (pts (xy 102.87 43.18) (xy 102.87 45.72))
     (stroke (width 0) (type default) (color 0 0 0 0))
@@
     (stroke (width 0) (type default) (color 0 0 0 0))
   )
-  (wire (pts (xy 63.5 109.22) (xy 67.31 109.22))
+  (wire (pts (xy 63.5 111.76) (xy 67.31 111.76))
     (stroke (width 0) (type default) (color 0 0 0 0))
   )
@@
     (effects (font (size 1.27 1.27)) (justify left bottom))
   )
+  (label "ALARM_EN" (at 214.63 104.14 0)
+    (effects (font (size 1.27 1.27)) (justify left bottom))
+  )
   (label "+5V" (at 20.32 144.78 0)
     (effects (font (size 1.27 1.27)) (justify left bottom))
@@
     (effects (font (size 1.27 1.27)) (justify left bottom))
   )
+  (label "GND" (at 179.07 109.22 0)
+    (effects (font (size 1.27 1.27)) (justify left bottom))
+  )
   (label "BLUE_IO" (at 67.31 124.46 0)
     (effects (font (size 1.27 1.27)) (justify left bottom))
   )
-  (label "RED_IO" (at 67.31 109.22 0)
+  (label "RED_IO" (at 67.31 111.76 0)
     (effects (font (size 1.27 1.27)) (justify left bottom))
   )
@@
     (effects (font (size 1.27 1.27)) (justify left bottom))
   )
+  (label "+3.3V" (at 179.07 99.06 0)
+    (effects (font (size 1.27 1.27)) (justify left bottom))
+  )
   (label "BLUE_IO" (at 140.97 43.18 0)
     (effects (font (size 1.27 1.27)) (justify left bottom))
   )
   (label "IR_D" (at 223.52 44.45 0)
+    (effects (font (size 1.27 1.27)) (justify left bottom))
+  )
+  (label "ALARM_EN" (at 67.31 109.22 0)
     (effects (font (size 1.27 1.27)) (justify left bottom))
   )
@@
     (pin "2")
   )
+  (symbol (lib_id "Switch:SW_SPDT") (at 203.2 104.14 180) (unit 1)
+    (in_bom yes) (on_board yes) (fields_autoplaced)
+    (property "Reference" "SW?" (id 0) (at 203.2 96.52 0))
+    (property "Value" "SW_SPDT" (id 1) (at 203.2 99.06 0))
+    (property "Footprint" "MattisLib:SS 13PLP" (id 2) (at 203.2 104.14 0)
+      (effects (font (size 1.27 1.27)) hide)
+    )
+    (property "Datasheet" "~" (id 3) (at 203.2 104.14 0)
+      (effects (font (size 1.27 1.27)) hide)
+    )
+    (pin "1")
+    (pin "2")
+    (pin "3")
+  )
   (symbol (lib_id "Transistor_FET:TSM2302CX") (at 83.82 45.72 0) (unit 1)
     (in_bom yes) (on_board yes) (fields_autoplaced)
@@
     (pin "2")
     (pin "3")
+  )
+  (symbol (lib_id "Device:R") (at 190.5 99.06 90) (unit 1)
+    (in_bom yes) (on_board yes) (fields_autoplaced)
+    (property "Reference" "R?" (id 0) (at 190.5 92.71 90))
+    (property "Value" "10k" (id 1) (at 190.5 95.25 90))
+    (property "Footprint" "Resistor_SMD:R_0805_2012Metric" (id 2) (at 190.5 100.838 90)
+      (effects (font (size 1.27 1.27)) hide)
+    )
+    (property "Datasheet" "~" (id 3) (at 190.5 99.06 0)
+      (effects (font (size 1.27 1.27)) hide)
+    )
+    (pin "1")
+    (pin "2")
   )
   (symbol (lib_id "power:GND") (at 22.86 36.83 0) (unit 1)
@@
     (pin "2")
     (pin "3")
+  )
+  (symbol (lib_id "Device:R") (at 190.5 109.22 90) (unit 1)
+    (in_bom yes) (on_board yes) (fields_autoplaced)
+    (property "Reference" "R?" (id 0) (at 190.5 102.87 90))
+    (property "Value" "10k" (id 1) (at 190.5 105.41 90))
+    (property "Footprint" "Resistor_SMD:R_0805_2012Metric" (id 2) (at 190.5 110.998 90)
+      (effects (font (size 1.27 1.27)) hide)
+    )
+    (property "Datasheet" "~" (id 3) (at 190.5 109.22 0)
+      (effects (font (size 1.27 1.27)) hide)
+    )
+    (pin "1")
+    (pin "2")
   )
   (symbol (lib_id "Transistor_FET:TSM2302CX") (at 160.02 45.72 0) (unit 1)
@@
       (reference "R6") (unit 1) (value "5k6") (footprint "Resistor_SMD:R_0805_2012Metric")
     )
+    (path "/8a4a253d-c044-4c3b-8069-83c4312624ae"
+      (reference "R?") (unit 1) (value "10k") (footprint "Resistor_SMD:R_0805_2012Metric")
+    )
+    (path "/b38d633a-556b-440a-b1e9-5d7324194536"
+      (reference "R?") (unit 1) (value "10k") (footprint "Resistor_SMD:R_0805_2012Metric")
+    )
+    (path "/73023868-ccbd-4c2d-8813-1d0b1e1e9efc"
+      (reference "SW?") (unit 1) (value "SW_SPDT") (footprint "MattisLib:SS 13PLP")
+    )
     (path "/100708ee-4125-4f5a-b2e4-ac3378e710a6"

Commit message: Refactor
Parts:
- gave numbers to parts that had none: 3
Changed lines of the file:
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@@
   (symbol (lib_id "Switch:SW_SPDT") (at 203.2 104.14 180) (unit 1)
     (in_bom yes) (on_board yes) (fields_autoplaced)
-    (property "Reference" "SW?" (id 0) (at 203.2 96.52 0))
+    (property "Reference" "SW1" (id 0) (at 203.2 96.52 0))
     (property "Value" "SW_SPDT" (id 1) (at 203.2 99.06 0))
     (property "Footprint" "MattisLib:SS 13PLP" (id 2) (at 203.2 104.14 0)
@@
   (symbol (lib_id "Device:R") (at 190.5 99.06 90) (unit 1)
     (in_bom yes) (on_board yes) (fields_autoplaced)
-    (property "Reference" "R?" (id 0) (at 190.5 92.71 90))
+    (property "Reference" "R7" (id 0) (at 190.5 92.71 90))
     (property "Value" "10k" (id 1) (at 190.5 95.25 90))
     (property "Footprint" "Resistor_SMD:R_0805_2012Metric" (id 2) (at 190.5 100.838 90)
@@
   (symbol (lib_id "Device:R") (at 190.5 109.22 90) (unit 1)
     (in_bom yes) (on_board yes) (fields_autoplaced)
-    (property "Reference" "R?" (id 0) (at 190.5 102.87 90))
+    (property "Reference" "R8" (id 0) (at 190.5 102.87 90))
     (property "Value" "10k" (id 1) (at 190.5 105.41 90))
     (property "Footprint" "Resistor_SMD:R_0805_2012Metric" (id 2) (at 190.5 110.998 90)
@@
     )
     (path "/8a4a253d-c044-4c3b-8069-83c4312624ae"
-      (reference "R?") (unit 1) (value "10k") (footprint "Resistor_SMD:R_0805_2012Metric")
+      (reference "R7") (unit 1) (value "10k") (footprint "Resistor_SMD:R_0805_2012Metric")
     )
     (path "/b38d633a-556b-440a-b1e9-5d7324194536"
-      (reference "R?") (unit 1) (value "10k") (footprint "Resistor_SMD:R_0805_2012Metric")
+      (reference "R8") (unit 1) (value "10k") (footprint "Resistor_SMD:R_0805_2012Metric")
     )
     (path "/73023868-ccbd-4c2d-8813-1d0b1e1e9efc"
-      (reference "SW?") (unit 1) (value "SW_SPDT") (footprint "MattisLib:SS 13PLP")
+      (reference "SW1") (unit 1) (value "SW_SPDT") (footprint "MattisLib:SS 13PLP")
     )
     (path "/100708ee-4125-4f5a-b2e4-ac3378e710a6"
